File: schematics/d11toy2d.brd (EAGLE design)
At the start: 16.7 x 29.2 mm, 17 parts, among them J1 usb, J2 strip, SW1 SPST_TACT-KMR2, U1 SAMD11, U2 74AHC1G125, U3 XC6206P332MR-G-SOT23

Commit message: more experiments
Parts:
- removed R1: 500, SparkFun-Passives:0603-RES
- added VIN: (no value), SparkFun-Connectors:1X02
- D2: value (none) -> boot
- moved SW1 12.2 mm to (15.0, 12.4)
- moved C2 6.86 mm to (2.54, 15.7), turned to 90 degrees
- moved U3 6.40 mm to (2.03, 12.4), turned to 90 degrees
- moved R3 1.48 mm to (14.7, 17.3), turned to 0 degrees
- moved U1 1.14 mm to (8.64, 12.4)
- moved C1 1.05 mm to (4.83, 7.11), turned to 0 degrees
- moved J2 1.02 mm to (4.57, 27.4)
- moved C3 0.57 mm to (10.9, 7.11), turned to 0 degrees
- moved R4 0.51 mm to (14.0, 23.9)
- moved D1 0.51 mm to (14.5, 5.33)
- moved R2 0.51 mm to (14.5, 7.11)
- moved U2 0.25 mm to (14.0, 20.3)
Connections:
- removed net N$2: R1.2, SW1.2, SW1.4
- removed net N$4: U2.1
- net 5V: now also VIN.2
- net GND: now also U2.1, VIN.1
- net N$3: now also C4.1
- net RES: now also SW1.2, SW1.4; no longer R1.1
Routing:
- net RES: track 6.64 -> 14.9 mm
- net N$2: track 5.97 -> 0.00 mm
- net +3V3: track 17.8 -> 13.8 mm
- net N$5: track 15.0 -> 17.4 mm
- net N$3: track 2.37 -> 4.17 mm
- net GND: track 9.78 -> 8.00 mm
- net PA02: track 3.11 -> 4.29 mm
- net LEDDO: track 10.2 -> 11.2 mm
Other:
- board text added: "d11toy2d"
- board text removed: "d11toy2b"
