File: schematics/d11toy2d.sch (EAGLE design)
At the start: 17 parts, among them J1 usb, J2 strip, SW1 SPST_TACT-KMR2, U1 SAMD11, U2 74AHC1G125, U3 XC6206P332MR-G-SOT23

Commit message: more experiments
Parts:
- removed R1: 500, SparkFun-Passives:RESISTOR0603-RES
- added VIN: (no value), SparkFun-Connectors:M02PTH
- D2: value (none) -> boot
Connections:
- removed net N$2: R1.2, SW1.S, SW1.S1
- removed net N$4: U2./OE
- net 5V: now also VIN.2
- net GND: now also U2./OE, VIN.1
- net N$3: now also C4.1
- net RES: now also SW1.S, SW1.S1; no longer R1.1
