File: schematics/d11toy4.brd (EAGLE design)
At the start: 16.7 x 29.2 mm, 15 parts, among them J1 usb, J2 strip, SW1 SPST_TACT-KMR2, U3 XC6206P332MR-G-SOT23

Commit message: more experiments
Parts:
- added C5: 100n, SparkFun-Capacitors:0603-CAP
- added D2: LED, SparkFun-LED:LED-0603
- added LED2: WS2812B5050, adafruit:WS2812B
- D1: value LED -> (none); device SparkFun-LED:LED-0603 -> SparkFun-DiscreteSemi:SOD523
- moved R1 16.7 mm to (15.5, 6.10), turned to 270 degrees
- moved R2 14.1 mm to (1.52, 13.5), flipped to the bottom
- moved SW1 12.8 mm to (8.38, 1.78), turned to 180 degrees
- moved D1 11.6 mm to (1.78, 11.9), turned to 270 degrees
- moved R4 9.48 mm to (15.5, 10.4), turned to 270 degrees
- moved LED1 8.92 mm to (11.4, 11.9), turned to 90 degrees
- moved R5 8.23 mm to (15.5, 13.7), turned to 90 degrees
- moved J2 7.62 mm to (4.57, 18.8)
- moved C4 7.52 mm to (5.33, 13.5), flipped to the bottom
- moved C2 7.50 mm to (9.65, 6.10), turned to 90 degrees
- moved C1 4.50 mm to (1.52, 6.10), turned to 270 degrees
- moved C3 3.54 mm to (7.11, 6.10), turned to 90 degrees
- moved U2 2.74 mm to (7.87, 8.89), flipped to the bottom
- moved U3 0.76 mm to (2.79, 6.86), flipped to the bottom, turned to 270 degrees
- flipped J1 to the bottom
Connections:
- new net N$3: LED1.2-DOUT, LED2.4-DIN
- new net N$4: C4.1, C5.1, D1.C, LED1.1-VDD, LED2.1-VDD
- net 5V: now also D1.A; no longer C4.1, LED1.1-VDD
- net GND: now also C5.2, D2.C, LED2.3-GND; no longer D1.C
- net LEDDAT: now also U2.4
- net LEDDO: now also LED2.2-DOUT; no longer LED1.2-DOUT
- net N$1: now also D2.A; no longer D1.A
Routing:
- net GND: track 0.00 -> 38.4 mm, vias 0 -> 2
- net 5V: track 0.00 -> 36.3 mm, vias 0 -> 2
- net N$4: track 0.00 -> 25.0 mm, vias 0 -> 2
- net LEDDAT: track 0.00 -> 18.0 mm, vias 0 -> 1
- net LEDDO: track 0.00 -> 17.7 mm
- net +3V3: track 0.00 -> 11.0 mm, vias 0 -> 1
- net N$2: track 0.00 -> 10.6 mm
- net PA02: track 0.00 -> 8.16 mm
- net RES: track 0.00 -> 6.28 mm, vias 0 -> 1
- net N$3: track 0.00 -> 6.06 mm
- net USBDM: track 0.00 -> 2.95 mm
- net USBDP: track 0.00 -> 2.89 mm
- net N$5: track 0.00 -> 2.49 mm
- net N$1: track 0.00 -> 1.79 mm
- added copper zone on layer 16, net GND
- removed copper zone on layer 1, net GND
Other:
- board size 16.7 x 29.2 mm -> 16.7 x 20.3 mm
- board text added: "d11toy4"
- board text removed: "d11toy2"
